File: ECE411.kicad_sch (KiCad schematic)
At the start: 8 parts, among them J1-ToPump Conn_01x02_Female, J2-ToMoistSense Conn_01x02_Female, Q1 2N7000

Commit message: Add files via upload
Parts:
- removed Q1: 2N7000, Package_TO_SOT_THT:TO-92_Inline, symbol Transistor_FET:2N7000
- removed R1: 33, symbol Device:R
- added Q1: 2N7002, Package_TO_SOT_SMD:SOT-23, symbol Transistor_FET:2N7002
- added R2: 15 Ohm, Resistor_SMD:R_0402_1005Metric, symbol Device:R
- added R3: 220 Ohm, Resistor_SMD:R_0402_1005Metric, symbol Device:R
- Batt1: renamed from 4.5VBatt; value Battery -> 4.5 V Battery; footprint (none) -> TestPoint:TestPoint_Bridge_Pitch7.62mm_Drill1.3mm
- J1-ToPump1: renamed from J1-ToPump; footprint (none) -> TestPoint:TestPoint_Bridge_Pitch5.08mm_Drill1.3mm
- J2-ToMoistSense1: renamed from J2-ToMoistSense; footprint (none) -> TestPoint:TestPoint_Bridge_Pitch5.08mm_Drill1.3mm
- R1: footprint (none) -> Potentiometer_SMD:Potentiometer_Bourns_TC33X_Vertical
Connections:
- net at A1.4 (GND), Batt1.2 (-), DS1.16 (LED(-))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: now also R2.2
- net at J1-ToPump1.1 (Pin_1): now also Q1.3 (D)
- net at A1.26 (USB), Batt1.1 (+), DS1.1 (VSS)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: now also R3.1; no longer DS1.15 (LED(+))
- net at A1.12 (MOSI/IO18): now also DS1.6 (E); no longer DS1.11 (D4)
- net at A1.14 (RX/IO16): no longer DS1.13 (D6)
- net at A1.15 (TX/IO17): no longer DS1.12 (D5)
- net at A1.17 (SDA/IO23): no longer DS1.6 (E)
- net at A1.19 (A6/IO14): now also DS1.11 (D4)
- net at A1.20 (A7/IO32): now also DS1.12 (D5)
- net at A1.21 (A8/IO15): now also DS1.13 (D6); no longer DS1.14 (D7)
- net at A1.22 (A9/IO33): now also DS1.14 (D7)
- net at A1.5 (DAC2/A0): now also Q1.1 (G)
- new net: DS1.15 (LED(+)), R3.2
- new net: Q1.2 (S), R2.1
- no-connect marks 0 -> 21
