File: Schematic Files/KiCad/ECE411.kicad_sch (KiCad schematic)
At the start: 9 parts, among them J1-ToPump1 Conn_01x02_Female, J2-ToMoistSense1 Conn_01x02_Female, Q1 2N7002

Commit message: Add files via upload
Parts:
- Batt1: footprint TestPoint:TestPoint_Bridge_Pitch7.62mm_Drill1.3mm -> TestPoint:TestPoint_2Pads_Pitch5.08mm_Drill1.3mm
- J1-ToPump1, J2-ToMoistSense1: footprint TestPoint:TestPoint_Bridge_Pitch5.08mm_Drill1.3mm -> TestPoint:TestPoint_2Pads_Pitch5.08mm_Drill1.3mm
Changed lines of the file:
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@@
     (property "Reference" "J1-ToPump1" (id 0) (at 123.19 95.25 90))
     (property "Value" "Conn_01x02_Female" (id 1) (at 123.19 97.79 90))
-    (property "Footprint" "TestPoint:TestPoint_Bridge_Pitch5.08mm_Drill1.3mm" (id 2) (at 123.19 101.6 0)
+    (property "Footprint" "TestPoint:TestPoint_2Pads_Pitch5.08mm_Drill1.3mm" (id 2) (at 123.19 101.6 0)
       (effects (font (size 1.27 1.27)) hide)
     )
@@
     (property "Reference" "J2-ToMoistSense1" (id 0) (at 97.79 63.5 90))
     (property "Value" "Conn_01x02_Female" (id 1) (at 97.79 66.04 90))
-    (property "Footprint" "TestPoint:TestPoint_Bridge_Pitch5.08mm_Drill1.3mm" (id 2) (at 97.79 69.85 0)
+    (property "Footprint" "TestPoint:TestPoint_2Pads_Pitch5.08mm_Drill1.3mm" (id 2) (at 97.79 69.85 0)
       (effects (font (size 1.27 1.27)) hide)
     )
@@
     (property "Reference" "Batt1" (id 0) (at 159.639 137.16 90))
     (property "Value" "4.5 V Battery" (id 1) (at 159.639 139.7 90))
-    (property "Footprint" "TestPoint:TestPoint_Bridge_Pitch7.62mm_Drill1.3mm" (id 2) (at 158.496 144.78 90)
+    (property "Footprint" "TestPoint:TestPoint_2Pads_Pitch5.08mm_Drill1.3mm" (id 2) (at 158.496 144.78 90)
       (effects (font (size 1.27 1.27)) hide)
     )
@@
     )
     (path "/d2893233-9ea8-4931-bf6d-45c22dc272a5"
-      (reference "Batt1") (unit 1) (value "4.5 V Battery") (footprint "TestPoint:TestPoint_Bridge_Pitch7.62mm_Drill1.3mm")
+      (reference "Batt1") (unit 1) (value "4.5 V Battery") (footprint "TestPoint:TestPoint_2Pads_Pitch5.08mm_Drill1.3mm")
     )
     (path "/f53f9c9b-3369-42be-8ddc-556529932eef"
@@
     )
     (path "/243048db-0907-4805-9618-fbea523b1cd7"
-      (reference "J1-ToPump1") (unit 1) (value "Conn_01x02_Female") (footprint "TestPoint:TestPoint_Bridge_Pitch5.08mm_Drill1.3mm")
+      (reference "J1-ToPump1") (unit 1) (value "Conn_01x02_Female") (footprint "TestPoint:TestPoint_2Pads_Pitch5.08mm_Drill1.3mm")
     )
     (path "/78f7b647-2d0f-4843-a7b2-f34cbcc8cd8f"
-      (reference "J2-ToMoistSense1") (unit 1) (value "Conn_01x02_Female") (footprint "TestPoint:TestPoint_Bridge_Pitch5.08mm_Drill1.3mm")
+      (reference "J2-ToMoistSense1") (unit 1) (value "Conn_01x02_Female") (footprint "TestPoint:TestPoint_2Pads_Pitch5.08mm_Drill1.3mm")
     )
     (path "/bdc29a76-653b-4536-9c61-ee0ddc4c017a"
